File: hardware/eagle_files/rev0.1.sch (EAGLE design)
At the start: 66 parts, among them U1 AD8332ACPZ-R7, U2 AD8333ACPZ-REEL

Commit message: All traces routed
Parts:
- removed RST: 22-23-2031, con-molex:22-23-2031
- added RESET: (no value), SparkFun-Connectors:M03PTH
- ENABLE, PH10, PH11, PH12, PH13: value 22-23-2031 -> (none); device con-molex:22-23-2031 -> SparkFun-Connectors:M03PTH
- R9: device resistor:R-US_R0603 -> resistor:R-US_R1206
- renumbered C3 to C12, C4 to C24
Connections:
- net +5V: now also PH10.1, PH11.3, PH12.1, PH13.3, RESET.3; no longer PH10-1.S, PH11-3.S, PH12-1.S, PH13-3.S, RST-3.S
- net ENBL: now also ENABLE.2; no longer ENABLE-2.S
- net GND: now also ENABLE.3, PH10.3, PH11.1, PH12.3, PH13.1, RESET.1, U1.EP; no longer ENABLE-3.S, PH10-3.S, PH11-1.S, PH12-3.S, PH13-1.S, RST-1.S
- net N$11: now also RESET.2; no longer RST-2.S
- net PH10: now also PH10.2; no longer PH10-2.S
- net PH11: now also PH11.2; no longer PH11-2.S
- net PH12: now also PH12.2; no longer PH12-2.S
- net PH13: now also PH13.2; no longer PH13-2.S
- net VPOS: now also ENABLE.1; no longer ENABLE-1.S
